File: kicad-global/MS20-VCF.kicad_pcb (KiCad board)
At the start: 2 copper layers, 118 x 128.5 mm, 59 parts, among them J5 Power Input, J6 FilterCV1, J7 FilterIn1, J8 FilterOut1, Q1 BC559, Q2 BC559, SW1 Hpass/Lpass Switch, U1 LM13700, U2 TL072

Commit message: update footprint trimmer
Parts:
- C2, C3: value 10µ -> 10uF
- C6: value 10µF -> 10uF
- ResLv1: value 3.3k -> 10k; footprint Potentiometer_THT:Potentiometer_Bourns_3386C_Horizontal -> Potentiometer_THT:Potentiometer_Bourns_3386X_Horizontal
- ResVol1: footprint Potentiometer_THT:Potentiometer_Bourns_3386C_Horizontal -> Potentiometer_THT:Potentiometer_Bourns_3386X_Horizontal
- moved ResLv1 1.17 mm to (81.0, 44.2)
- moved ResVol1 1.17 mm to (81.0, 54.8)
Routing:
- net Net-(C1-Pad2): track 86.2 -> 84.5 mm
- net Net-(D2-Pad2): track 23.7 -> 22.1 mm
- net Net-(D6-Pad1): track 69.0 -> 67.8 mm
