File: kicad-global/MS20-VCF.kicad_sch (KiCad schematic)
At the start: 59 parts, among them J5 Power Input, J6 FilterCV1, J7 FilterIn1, J8 FilterOut1, Q1 BC559, Q2 BC559, SW1 Hpass/Lpass Switch, U1 LM13700, U2 TL072

Commit message: add details and fix issues
Parts:
- C2, C3: value 10µ -> 10uF; Comment  (none) -> Electrolytic cap
- C6: value 10µF -> 10uF; Comment  (none) -> Electrolytic cap
- CUTCV1: Comment  (none) -> Use a small one (trimmer type)
- Q1, Q2: Comment  (none) -> substitute BC558
- ResLv1, ResVol1: Comment  (none) -> variable resistor
Changed lines of the file:
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@@
     (pin "15")
     (pin "16")
-    (pin "10")
-    (pin "9")
+  )
+  (symbol (lib_id "Amplifier_Operational:LM13700") (at 96.52 52.07 0) (unit 3)
+    (in_bom yes) (on_board yes)
+    (property "Reference" "U1" (id 0) (at 96.52 42.7482 0))
+    (property "Value" "LM13700" (id 1) (at 96.52 45.0596 0))
+    (property "Footprint" "Package_SO:SOIC-16_3.9x9.9mm_P1.27mm" (id 2) (at 88.9 51.435 0)
+      (effects (font (size 1.27 1.27)) hide)
+    )
+    (property "Datasheet" "http://www.ti.com/lit/ds/symlink/lm13700.pdf" (id 3) (at 88.9 51.435 0)
+      (effects (font (size 1.27 1.27)) hide)
+    )
     (pin "1")
     (pin "2")
@@
     (pin "4")
     (pin "5")
-    (pin "7")
-    (pin "8")
-    (pin "11")
-    (pin "6")
-  )
-  (symbol (lib_id "Amplifier_Operational:LM13700") (at 96.52 52.07 0) (unit 3)
-    (in_bom yes) (on_board yes)
-    (property "Reference" "U1" (id 0) (at 96.52 42.7482 0))
-    (property "Value" "LM13700" (id 1) (at 96.52 45.0596 0))
-    (property "Footprint" "Package_SO:SOIC-16_3.9x9.9mm_P1.27mm" (id 2) (at 88.9 51.435 0)
-      (effects (font (size 1.27 1.27)) hide)
-    )
-    (property "Datasheet" "http://www.ti.com/lit/ds/symlink/lm13700.pdf" (id 3) (at 88.9 51.435 0)
-      (effects (font (size 1.27 1.27)) hide)
-    )
-    (pin "12")
-    (pin "13")
-    (pin "14")
-    (pin "15")
-    (pin "16")
-    (pin "10")
-    (pin "9")
-    (pin "1")
-    (pin "2")
-    (pin "3")
-    (pin "4")
-    (pin "5")
-    (pin "7")
-    (pin "8")
-    (pin "11")
-    (pin "6")
   )
   (symbol (lib_id "Amplifier_Operational:LM13700") (at 190.5 52.07 0) (unit 2)
@@
       (effects (font (size 1.27 1.27)) hide)
     )
-    (pin "12")
-    (pin "13")
-    (pin "14")
-    (pin "15")
-    (pin "16")
     (pin "10")
     (pin "9")
-    (pin "1")
-    (pin "2")
-    (pin "3")
-    (pin "4")
-    (pin "5")
-    (pin "7")
-    (pin "8")
-    (pin "11")
-    (pin "6")
   )
   (symbol (lib_id "Amplifier_Operational:LM13700") (at 125.73 52.07 0) (unit 4)
@@
       (effects (font (size 1.27 1.27)) hide)
     )
-    (pin "12")
-    (pin "13")
-    (pin "14")
-    (pin "15")
-    (pin "16")
-    (pin "10")
-    (pin "9")
-    (pin "1")
-    (pin "2")
-    (pin "3")
-    (pin "4")
-    (pin "5")
     (pin "7")
     (pin "8")
-    (pin "11")
-    (pin "6")
   )
   (symbol (lib_id "Amplifier_Operational:TL072") (at 193.04 78.74 180) (unit 1)
@@
     (pin "2")
     (pin "3")
+  )
+  (symbol (lib_id "Amplifier_Operational:TL072") (at 138.43 100.33 180) (unit 2)
+    (in_bom yes) (on_board yes)
+    (property "Reference" "U2" (id 0) (at 137.16 104.14 0))
+    (property "Value" "TL072" (id 1) (at 137.16 106.68 0))
+    (property "Footprint" "Package_DIP:DIP-8_W7.62mm_Socket" (id 2) (at 138.43 100.33 0)
+      (effects (font (size 1.27 1.27)) hide)
+    )
+    (property "Datasheet" "http://www.ti.com/lit/ds/symlink/tl071.pdf" (id 3) (at 138.43 100.33 0)
+      (effects (font (size 1.27 1.27)) hide)
+    )
     (pin "5")
     (pin "6")
     (pin "7")
-    (pin "4")
-    (pin "8")
-  )
-  (symbol (lib_id "Amplifier_Operational:TL072") (at 138.43 100.33 180) (unit 2)
-    (in_bom yes) (on_board yes)
-    (property "Reference" "U2" (id 0) (at 137.16 104.14 0))
-    (property "Value" "TL072" (id 1) (at 137.16 106.68 0))
-    (property "Footprint" "Package_DIP:DIP-8_W7.62mm_Socket" (id 2) (at 138.43 100.33 0)
-      (effects (font (size 1.27 1.27)) hide)
-    )
-    (property "Datasheet" "http://www.ti.com/lit/ds/symlink/tl071.pdf" (id 3) (at 138.43 100.33 0)
-      (effects (font (size 1.27 1.27)) hide)
-    )
-    (pin "1")
-    (pin "2")
-    (pin "3")
-    (pin "5")
-    (pin "6")
-    (pin "7")
-    (pin "4")
-    (pin "8")
   )
   (symbol (lib_id "Device:R") (at 76.2 54.61 90) (unit 1)
@@
     (in_bom yes) (on_board yes)
     (property "Reference" "C6" (id 0) (at 207.01 48.133 90))
-    (property "Value" "10µF" (id 1) (at 207.01 50.4444 90))
+    (property "Value" "10uF" (id 1) (at 207.01 50.4444 90))
     (property "Footprint" "Capacitor_THT:CP_Radial_D5.0mm_P2.00mm" (id 2) (at 203.2 55.5752 0)
       (effects (font (size 1.27 1.27)) hide)
     )
     (property "Datasheet" "~" (id 3) (at 207.01 54.61 0)
+      (effects (font (size 1.27 1.27)) hide)
+    )
+    (property "Comment " "Electrolytic cap" (id 4) (at 207.01 54.61 0)
       (effects (font (size 1.27 1.27)) hide)
     )
@@
       (effects (font (size 1.27 1.27)) hide)
     )
+    (property "Comment " "Use a small one (trimmer type)" (id 4) (at 167.64 123.19 0)
+      (effects (font (size 1.27 1.27)) hide)
+    )
     (pin "1")
     (pin "2")
@@
       (effects (font (size 1.27 1.27)) (justify left) hide)
     )
+    (property "Comment " "substitute BC558" (id 4) (at 101.6 114.3 0)
+      (effects (font (size 1.27 1.27)) hide)
+    )
     (pin "1")
     (pin "2")
@@
     (property "Datasheet" "https://www.onsemi.com/pub/Collateral/BC556BTA-D.pdf" (id 3) (at 120.65 114.3 0)
       (effects (font (size 1.27 1.27)) (justify left) hide)
+    )
+    (property "Comment " "substitute BC558" (id 4) (at 120.65 114.3 0)
+      (effects (font (size 1.27 1.27)) hide)
     )
     (pin "1")
@@
       (effects (font (size 1.27 1.27)) (justify left))
     )
-    (property "Value" "10µ" (id 1) (at 138.2014 171.323 0)
+    (property "Value" "10uF" (id 1) (at 138.2014 171.323 0)
       (effects (font (size 1.27 1.27)) (justify left))
     )
@@
       (effects (font (size 1.27 1.27)) hide)
     )
+    (property "Comment " "Electrolytic cap" (id 4) (at 135.89 170.18 0)
+      (effects (font (size 1.27 1.27)) hide)
+    )
     (pin "1")
     (pin "2")
@@
       (effects (font (size 1.27 1.27)) (justify left))
     )
-    (property "Value" "10µ" (id 1) (at 138.2014 185.293 0)
+    (property "Value" "10uF" (id 1) (at 138.2014 185.293 0)
       (effects (font (size 1.27 1.27)) (justify left))
     )
@@
     )
     (property "Datasheet" "~" (id 3) (at 135.89 184.15 0)
+      (effects (font (size 1.27 1.27)) hide)
+    )
+    (property "Comment " "Electrolytic cap" (id 4) (at 135.89 184.15 0)
       (effects (font (size 1.27 1.27)) hide)
     )
@@
       (effects (font (size 1.27 1.27)) hide)
     )
+    (property "Comment " "variable resistor" (id 4) (at 195.58 93.98 0)
+      (effects (font (size 1.27 1.27)) hide)
+    )
     (pin "1")
     (pin "2")
@@
       (effects (font (size 1.27 1.27)) hide)
     )
-    (pin "12")
-    (pin "13")
-    (pin "14")
-    (pin "15")
-    (pin "16")
-    (pin "10")
-    (pin "9")
-    (pin "1")
-    (pin "2")
-    (pin "3")
-    (pin "4")
-    (pin "5")
-    (pin "7")
-    (pin "8")
     (pin "11")
     (pin "6")
@@
       (effects (font (size 1.27 1.27)) hide)
     )
-    (pin "1")
-    (pin "2")
-    (pin "3")
-    (pin "5")
-    (pin "6")
-    (pin "7")
     (pin "4")
     (pin "8")
@@
     )
     (property "Datasheet" "~" (id 3) (at 176.53 93.98 0)
+      (effects (font (size 1.27 1.27)) hide)
+    )
+    (property "Comment " "variable resistor" (id 4) (at 176.53 93.98 0)
       (effects (font (size 1.27 1.27)) hide)
     )
@@
     )
     (path "/00000000-0000-0000-0000-0000614ba8d1"
-      (reference "C2") (unit 1) (value "10µ") (footprint "Capacitor_THT:CP_Radial_D5.0mm_P2.00mm")
+      (reference "C2") (unit 1) (value "10uF") (footprint "Capacitor_THT:CP_Radial_D5.0mm_P2.00mm")
     )
     (path "/00000000-0000-0000-0000-0000614ba8d7"
-      (reference "C3") (unit 1) (value "10µ") (footprint "Capacitor_THT:CP_Radial_D5.0mm_P2.00mm")
+      (reference "C3") (unit 1) (value "10uF") (footprint "Capacitor_THT:CP_Radial_D5.0mm_P2.00mm")
     )
     (path "/00000000-0000-0000-0000-0000603fad90"
@@
     )
     (path "/00000000-0000-0000-0000-000060355101"
-      (reference "C6") (unit 1) (value "10µF") (footprint "Capacitor_THT:CP_Radial_D5.0mm_P2.00mm")
+      (reference "C6") (unit 1) (value "10uF") (footprint "Capacitor_THT:CP_Radial_D5.0mm_P2.00mm")
     )
     (path "/473533f9-4d59-4ee6-9ea8-a3401341479e"

Commit message: update footprint trimmer
Parts:
- ResLv1: value 3.3k -> 10k; footprint Potentiometer_THT:Potentiometer_Bourns_3386C_Horizontal -> Potentiometer_THT:Potentiometer_Bourns_3386X_Horizontal
- ResVol1: footprint Potentiometer_THT:Potentiometer_Bourns_3386C_Horizontal -> Potentiometer_THT:Potentiometer_Bourns_3386X_Horizontal
- SW1: Comment  DPDT Switch, On-Off-On -> DPDT Switch, On-On
Changed lines of the file:
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@@
       (effects (font (size 1.27 1.27)) hide)
     )
-    (property "Comment " "DPDT Switch, On-Off-On " (id 4) (at 48.26 77.47 0)
+    (property "Comment " "DPDT Switch, On-On " (id 4) (at 48.26 77.47 0)
       (effects (font (size 1.27 1.27)) hide)
     )
@@
       (effects (font (size 1.27 1.27)) (justify right))
     )
-    (property "Value" "3.3k" (id 1) (at 193.04 93.98 90)
+    (property "Value" "10k" (id 1) (at 193.04 93.98 90)
       (effects (font (size 1.27 1.27)) (justify right))
     )
-    (property "Footprint" "Potentiometer_THT:Potentiometer_Bourns_3386C_Horizontal" (id 2) (at 195.58 93.98 0)
+    (property "Footprint" "Potentiometer_THT:Potentiometer_Bourns_3386X_Horizontal" (id 2) (at 195.58 93.98 0)
       (effects (font (size 1.27 1.27)) hide)
     )
@@
       (effects (font (size 1.27 1.27)) (justify right))
     )
-    (property "Footprint" "Potentiometer_THT:Potentiometer_Bourns_3386C_Horizontal" (id 2) (at 176.53 93.98 0)
+    (property "Footprint" "Potentiometer_THT:Potentiometer_Bourns_3386X_Horizontal" (id 2) (at 176.53 93.98 0)
       (effects (font (size 1.27 1.27)) hide)
     )
@@
     )
     (path "/00000000-0000-0000-0000-0000615804ec"
-      (reference "ResLv1") (unit 1) (value "3.3k") (footprint "Potentiometer_THT:Potentiometer_Bourns_3386C_Horizontal")
+      (reference "ResLv1") (unit 1) (value "10k") (footprint "Potentiometer_THT:Potentiometer_Bourns_3386X_Horizontal")
     )
     (path "/00000000-0000-0000-0000-0000616e3eb9"
-      (reference "ResVol1") (unit 1) (value "10k") (footprint "Potentiometer_THT:Potentiometer_Bourns_3386C_Horizontal")
+      (reference "ResVol1") (unit 1) (value "10k") (footprint "Potentiometer_THT:Potentiometer_Bourns_3386X_Horizontal")
     )
     (path "/00000000-0000-0000-0000-000060338cd7"

Commit message: update footprint for trimmer
Parts:
- ResLv1, ResVol1: footprint Potentiometer_THT:Potentiometer_Bourns_3386X_Horizontal -> Potentiometer_THT:Potentiometer_Bourns_3386C_Horizontal
Changed lines of the file:
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@@
     (pin "15")
     (pin "16")
+    (pin "10")
+    (pin "9")
+    (pin "1")
+    (pin "2")
+    (pin "3")
+    (pin "4")
+    (pin "5")
+    (pin "7")
+    (pin "8")
+    (pin "11")
+    (pin "6")
   )
   (symbol (lib_id "Amplifier_Operational:LM13700") (at 96.52 52.07 0) (unit 3)
@@
       (effects (font (size 1.27 1.27)) hide)
     )
+    (pin "12")
+    (pin "13")
+    (pin "14")
+    (pin "15")
+    (pin "16")
+    (pin "10")
+    (pin "9")
     (pin "1")
     (pin "2")
@@
     (pin "4")
     (pin "5")
+    (pin "7")
+    (pin "8")
+    (pin "11")
+    (pin "6")
   )
   (symbol (lib_id "Amplifier_Operational:LM13700") (at 190.5 52.07 0) (unit 2)
@@
       (effects (font (size 1.27 1.27)) hide)
     )
+    (pin "12")
+    (pin "13")
+    (pin "14")
+    (pin "15")
+    (pin "16")
     (pin "10")
     (pin "9")
+    (pin "1")
+    (pin "2")
+    (pin "3")
+    (pin "4")
+    (pin "5")
+    (pin "7")
+    (pin "8")
+    (pin "11")
+    (pin "6")
   )
   (symbol (lib_id "Amplifier_Operational:LM13700") (at 125.73 52.07 0) (unit 4)
@@
       (effects (font (size 1.27 1.27)) hide)
     )
+    (pin "12")
+    (pin "13")
+    (pin "14")
+    (pin "15")
+    (pin "16")
+    (pin "10")
+    (pin "9")
+    (pin "1")
+    (pin "2")
+    (pin "3")
+    (pin "4")
+    (pin "5")
     (pin "7")
     (pin "8")
+    (pin "11")
+    (pin "6")
   )
   (symbol (lib_id "Amplifier_Operational:TL072") (at 193.04 78.74 180) (unit 1)
@@
     (pin "2")
     (pin "3")
+    (pin "5")
+    (pin "6")
+    (pin "7")
+    (pin "4")
+    (pin "8")
   )
   (symbol (lib_id "Amplifier_Operational:TL072") (at 138.43 100.33 180) (unit 2)
@@
       (effects (font (size 1.27 1.27)) hide)
     )
+    (pin "1")
+    (pin "2")
+    (pin "3")
     (pin "5")
     (pin "6")
     (pin "7")
+    (pin "4")
+    (pin "8")
   )
   (symbol (lib_id "Device:R") (at 76.2 54.61 90) (unit 1)
@@
       (effects (font (size 1.27 1.27)) (justify right))
     )
-    (property "Footprint" "Potentiometer_THT:Potentiometer_Bourns_3386X_Horizontal" (id 2) (at 195.58 93.98 0)
+    (property "Footprint" "Potentiometer_THT:Potentiometer_Bourns_3386C_Horizontal" (id 2) (at 195.58 93.98 0)
       (effects (font (size 1.27 1.27)) hide)
     )
@@
       (effects (font (size 1.27 1.27)) hide)
     )
+    (pin "12")
+    (pin "13")
+    (pin "14")
+    (pin "15")
+    (pin "16")
+    (pin "10")
+    (pin "9")
+    (pin "1")
+    (pin "2")
+    (pin "3")
+    (pin "4")
+    (pin "5")
+    (pin "7")
+    (pin "8")
     (pin "11")
     (pin "6")
@@
       (effects (font (size 1.27 1.27)) hide)
     )
+    (pin "1")
+    (pin "2")
+    (pin "3")
+    (pin "5")
+    (pin "6")
+    (pin "7")
     (pin "4")
     (pin "8")
@@
       (effects (font (size 1.27 1.27)) (justify right))
     )
-    (property "Footprint" "Potentiometer_THT:Potentiometer_Bourns_3386X_Horizontal" (id 2) (at 176.53 93.98 0)
+    (property "Footprint" "Potentiometer_THT:Potentiometer_Bourns_3386C_Horizontal" (id 2) (at 176.53 93.98 0)
       (effects (font (size 1.27 1.27)) hide)
     )
@@
     )
     (path "/00000000-0000-0000-0000-0000615804ec"
-      (reference "ResLv1") (unit 1) (value "10k") (footprint "Potentiometer_THT:Potentiometer_Bourns_3386X_Horizontal")
+      (reference "ResLv1") (unit 1) (value "10k") (footprint "Potentiometer_THT:Potentiometer_Bourns_3386C_Horizontal")
     )
     (path "/00000000-0000-0000-0000-0000616e3eb9"
-      (reference "ResVol1") (unit 1) (value "10k") (footprint "Potentiometer_THT:Potentiometer_Bourns_3386X_Horizontal")
+      (reference "ResVol1") (unit 1) (value "10k") (footprint "Potentiometer_THT:Potentiometer_Bourns_3386C_Horizontal")
     )
     (path "/00000000-0000-0000-0000-000060338cd7"

Commit message: update repo organization
Other:
- company: (none) -> Bleep Sound
- title: (none) -> MS20 VCF
