File: fabrication/front/MS20-VCF.kicad_pcb (KiCad board)
At the start: 2 copper layers, 50 x 128.5 mm, 4 parts

Commit message: update to v1.2 on silkscreen
Other:
- board text added: "MS-20 VCF Face plate V1.2 BleepSound 2023"
- board text removed: "MS-20 VCF Face plate V1.1 BleepSound 2022"
Changed lines of the file:
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@@
       (drillshape 0)
       (scaleselection 1)
-      (outputdirectory "gerber/")
+      (outputdirectory "")
     )
   )
@@
   (gr_line (start 123.8 30.65) (end 123.8 32.35) (layer "F.SilkS") (width 0.12))
   (gr_line (start 117.5 86.5) (end 114.5 86.5) (layer "F.SilkS") (width 0.12))
-  (gr_arc (start 120 60) (mid 128.066778 34.359916) (end 135.889781 60.075425) (layer "F.SilkS") (width 0.12))
+  (gr_arc (start 120 60) (mid 128.066776 34.359917) (end 135.889781 60.075425) (layer "F.SilkS") (width 0.12))
   (gr_line (start 111.153553 59) (end 108.153553 59) (layer "F.SilkS") (width 0.12))
   (gr_arc (start 123.5 55) (mid 128 40.462851) (end 132.5 55) (layer "F.SilkS") (width 0.12))
@@
   (gr_arc (start 114 87) (mid 114.146447 86.646447) (end 114.5 86.5) (layer "F.SilkS") (width 0.12))
   (gr_line (start 126 31.75) (end 125.2 32.35) (layer "F.SilkS") (width 0.12))
-  (gr_arc (start 117.346447 96) (mid 117.699998 96.146448) (end 117.846447 96.5) (layer "F.SilkS") (width 0.12))
+  (gr_arc (start 117.346447 96) (mid 117.699999 96.146448) (end 117.846447 96.5) (layer "F.SilkS") (width 0.12))
   (gr_line (start 130.15 99.7) (end 129.95 99.6) (layer "F.SilkS") (width 0.12))
   (gr_line (start 109.4 125.2) (end 109.3 125.2) (layer "F.SilkS") (width 0.12))
@@
     (effects (font (size 1.5 1.5) (thickness 0.3)) (justify mirror))
   )
-  (gr_text "MS-20 VCF\nFace plate\nV1.1 BleepSound\n2022" (at 128 31) (layer "B.SilkS")
+  (gr_text "MS-20 VCF\nFace plate\nV1.2 BleepSound\n2023" (at 128 31) (layer "B.SilkS")
     (effects (font (size 1 1) (thickness 0.15)) (justify mirror))
   )
-  (dimension (type aligned) (layer "Dwgs.User")
-    (pts (xy 103 26.5) (xy 128 26.5))
-    (height -2.5)
-    (gr_text "25,0000 mm" (at 115.5 22.85) (layer "Dwgs.User")
-      (effects (font (size 1 1) (thickness 0.15)))
-    )
-    (format (units 3) (units_format 1) (precision 4))
-    (style (thickness 0.1) (arrow_length 1.27) (text_position_mode 0) (extension_height 0.58642) (extension_offset 0.5) keep_text_aligned)
-  )
-  (dimension (type aligned) (layer "Dwgs.User")
-    (pts (xy 158 153.5) (xy 149 153.5))
-    (height -7.5)
-    (gr_text "9,0000 mm" (at 153.5 159.85) (layer "Dwgs.User")
-      (effects (font (size 1 1) (thickness 0.15)))
-    )
-    (format (units 3) (units_format 1) (precision 4))
-    (style (thickness 0.1) (arrow_length 1.27) (text_position_mode 0) (extension_height 0.58642) (extension_offset 0.5) keep_text_aligned)
-  )
   (via (at 110 136) (size 6.8) (drill 6) (layers "F.Cu" "B.Cu") (net 1))
